Commit message: Updated joint limits for joint_t to match our robot

File: motoman_mh5_support/urdf/mh5.urdf (robot description, URDF)
Before this commit: robot motoman_mh5, 7 links, 6 joints
Joints:
- joint joint_t: limit lower=-6.2831 upper=6.2831 effort=100 velocity=6.97 -> lower=-3.1 upper=3.1 effort=100 velocity=6.97
- joint joint_u: limit lower=-2.3736 upper=4.4506 effort=100 velocity=2.96 -> lower=-1.0122 upper=3.2218 effort=100 velocity=2.96

File: motoman_mh5_support/urdf/mh5_macro.xacro (robot description, xacro)
@@ -159,4 +159,9 @@
 			<limit lower="-2.1817" upper="2.1817" effort="100" velocity="3.48" />
 		</joint>
+    <!--
+      Our MH5 robot has joint limits for joint_t at -3.14 and 3.14 at lowest speeds.
+      If set higher, it will give pulse limit errors before.
+      We will set the limits for joint_t to -3.1 and 3.1 to be on the safe side.
+    -->
 		<joint name="${prefix}joint_t" type="revolute">
 			<parent link="${prefix}link_b"/>
@@ -164,5 +169,5 @@
 			<origin xyz="0.0510 0 0" rpy="0 0 0"/>
 			<axis xyz="-1 0 0" />
-			<limit lower="-6.2831" upper="6.2831" effort="100" velocity="6.97" />
+			<limit lower="-3.1" upper="3.1" effort="100" velocity="6.97" />
 		</joint>
 		<!-- end of joint list -->
